File: mqtt_wlan_bridge/schematic/mqtt_bridge/mqtt_bridge.kicad_sch (KiCad schematic)
At the start: 4 parts, among them J1 Conn_Coaxial, U1 RFM95W-868S2, U2 ESP32-DevKitC

Commit message: backup
Parts:
- J1: footprint (none) -> Connector_Coaxial:SMA_Amphenol_901-144_Vertical
Other:
- title: (none) -> MQTT_WLAN_Bridge
Changed lines of the file:
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@@
 (kicad_sch (version 20211123) (generator eeschema)
   (paper "A4")
+  (title_block
+    (title "MQTT_WLAN_Bridge")
+    (date "2023-02-23")
+    (rev "1.0")
+  )
   (junction (at 100.33 109.22) (diameter 0) (color 0 0 0 0)
   )
@@
       (effects (font (size 1.27 1.27)) (justify left))
     )
-    (property "Footprint" "" (id 2) (at 120.65 67.31 0)
-      (effects (font (size 1.27 1.27)) hide)
-    )
+    (property "Footprint" "Connector_Coaxial:SMA_Amphenol_901-144_Vertical" (id 2) (at 120.65 67.31 0)
+      (effects (font (size 1.27 1.27)) hide)
+    )
